Commit message: tune local cost

File: urdf/turtlebot3_burger_custom.urdf.xacro (robot description, xacro)
@@ -159,5 +159,5 @@
   </link>
  <joint name="camera_joint" type="fixed">
-<!--	<origin xyz="0.073 -0.011 0.084" rpy="0 0.349 0"/> -->
+<!--	<origin xyz="0.073 -0.011 0.084" rpy="0 0 0"/> -->
   <origin xyz="0.055 0.032 0.208" rpy="0 0 0"/>
     <parent link="base_link"/>
@@ -168,5 +168,4 @@
       <origin xyz="0.0 0.0 0.0" rpy="0 0 0"/>
       <geometry>
-        <box size="0.015 0.030 0.027"/>
       </geometry>
     </collision>

Commit message: reduce cost

File: urdf/turtlebot3_burger_custom.urdf.xacro (robot description, xacro)
@@ -159,5 +159,5 @@
   </link>
  <joint name="camera_joint" type="fixed">
-<!--	<origin xyz="0.073 -0.011 0.084" rpy="0 0 0"/> -->
+<!--	<origin xyz="0.073 -0.011 0.084" rpy="0 0.349 0"/> -->
   <origin xyz="0.055 0.032 0.208" rpy="0 0 0"/>
     <parent link="base_link"/>
@@ -168,4 +168,5 @@
       <origin xyz="0.0 0.0 0.0" rpy="0 0 0"/>
       <geometry>
+        <box size="0.015 0.030 0.027"/>
       </geometry>
     </collision>

Commit message: test graph slam

File: urdf/turtlebot3_burger_custom.urdf.xacro (robot description, xacro)
@@ -15,5 +15,5 @@
         <mesh filename="package://turtlebot3_description/meshes/bases/burger_base.stl" scale="0.001 0.001 0.001"/>
       </geometry>
-      <material name="light_black"/>
+      <material name="purple"/>
     </visual>
     <collision>

Commit message: test graph slam

File: urdf/turtlebot3_burger_custom.urdf.xacro (robot description, xacro)
@@ -15,5 +15,5 @@
         <mesh filename="package://turtlebot3_description/meshes/bases/burger_base.stl" scale="0.001 0.001 0.001"/>
       </geometry>
-      <material name="purple"/>
+      <material name="Gazebo/Purple"/>
     </visual>
     <collision>

Commit message: test graph slam

File: urdf/turtlebot3_burger_custom.urdf.xacro (robot description, xacro)
@@ -3,4 +3,7 @@
   <xacro:include filename="$(find ballast_sim)/urdf/common_properties.xacro"/>
   <xacro:include filename="$(find ballast_sim)/urdf/turtlebot3_burger_custom.gazebo.xacro"/>
+  <material name="purple">
+       <color rgba="0.77 0.76 0.89 1"/>
+      </material>
   <link name="base_footprint"/>
   <joint name="base_joint" type="fixed">
@@ -15,5 +18,5 @@
         <mesh filename="package://turtlebot3_description/meshes/bases/burger_base.stl" scale="0.001 0.001 0.001"/>
       </geometry>
-      <material name="Gazebo/Purple"/>
+      <material name="purple"/>
     </visual>
     <collision>
